File: ground station/pcb/kicad Project/estacion terrena.kicad_sch (KiCad schematic)
At the start: 14 parts, among them J1 Micro-usb_lora, J10 IDC_STLINK, J11 IDC_CANSAT, J2 Parte izquierda lora, J3 parte derecha lora, J4 Breakouy_micro_usb, J5 CARG_BAT_1_OUT, J6 CARG_BAT_1_IN, J7 POSITIVO_LED TESTIGO, J8 CARG_BAT_2_OUT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

Commit message: Actualización
Parts:
- added R2: 120, Resistor_THT:R_Axial_DIN0207_L6.3mm_D2.5mm_P10.16mm_Horizontal, symbol Device:R
- K1: footprint Relay_THT:Relay_1P1T_NO_10x24x18.8mm_Panasonic_ADW11xxxxW_THT -> Relay_THT:RELAY PANASONIC
- R1: value R -> 330
Connections:
- net at R1.2, SW1.1 (A): now also R2.1; no longer K1.1
- new net: K1.1, R2.2
Other:
- note added: "RELE CARGA/PROGRAMACION"
- note removed: "RELE_CARGA/PROGRAMACION"
Changed lines of the file:
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@@
   (junction (at 163.83 67.31) (diameter 0) (color 0 0 0 0)
   )
+  (junction (at 167.64 128.27) (diameter 0) (color 0 0 0 0)
+  )
   (junction (at 105.41 121.92) (diameter 0) (color 0 0 0 0)
-  )
-  (junction (at 167.64 128.27) (diameter 0) (color 0 0 0 0)
   )
   (no_connect (at 207.01 76.2))
@@
     (stroke (width 0) (type default) (color 0 0 0 0))
   )
-  (wire (pts (xy 167.64 128.27) (xy 180.34 128.27))
-    (stroke (width 0) (type default) (color 0 0 0 0))
-  )
   (wire (pts (xy 173.99 64.77) (xy 149.86 64.77))
     (stroke (width 0) (type default) (color 0 0 0 0))
@@
     (stroke (width 0) (type default) (color 0 0 0 0))
   )
+  (wire (pts (xy 177.8 128.27) (xy 180.34 128.27))
+    (stroke (width 0) (type default) (color 0 0 0 0))
+  )
   (polyline (pts (xy 87.63 50.8) (xy 88.9 50.8))
     (stroke (width 0) (type default) (color 0 0 0 0))
@@
     (stroke (width 0) (type default) (color 0 0 0 0))
   )
+  (wire (pts (xy 167.64 128.27) (xy 170.18 128.27))
+    (stroke (width 0) (type default) (color 0 0 0 0))
+  )
   (wire (pts (xy 96.52 124.46) (xy 114.3 124.46))
     (stroke (width 0) (type default) (color 0 0 0 0))
@@
     (stroke (width 0) (type default) (color 0 0 0 0))
   )
-  (text "RELE_CARGA/PROGRAMACION\n" (at 156.21 158.75 0)
+  (text "RELE CARGA/PROGRAMACION\n" (at 154.94 156.21 0)
     (effects (font (size 1.27 1.27)) (justify left bottom))
   )
@@
   )
   (symbol (lib_id "Device:R") (at 167.64 121.92 0) (unit 1)
-    (in_bom yes) (on_board yes) (fields_autoplaced)
+    (in_bom yes) (on_board yes)
     (property "Reference" "R1" (id 0) (at 170.18 120.6499 0)
       (effects (font (size 1.27 1.27)) (justify left))
     )
-    (property "Value" "R" (id 1) (at 170.18 123.1899 0)
+    (property "Value" "330" (id 1) (at 162.56 121.92 0)
       (effects (font (size 1.27 1.27)) (justify left))
     )
@@
     (pin "4")
   )
+  (symbol (lib_id "Device:R") (at 173.99 128.27 90) (unit 1)
+    (in_bom yes) (on_board yes) (fields_autoplaced)
+    (property "Reference" "R2" (id 0) (at 173.99 121.92 90))
+    (property "Value" "120" (id 1) (at 173.99 124.46 90))
+    (property "Footprint" "Resistor_THT:R_Axial_DIN0207_L6.3mm_D2.5mm_P10.16mm_Horizontal" (id 2) (at 173.99 130.048 90)
+      (effects (font (size 1.27 1.27)) hide)
+    )
+    (property "Datasheet" "~" (id 3) (at 173.99 128.27 0)
+      (effects (font (size 1.27 1.27)) hide)
+    )
+    (pin "1")
+    (pin "2")
+  )
   (symbol (lib_id "Switch:SW_DPDT_x2") (at 151.13 135.89 0) (unit 1)
     (in_bom yes) (on_board yes) (fields_autoplaced)
@@
       (effects (font (size 1.27 1.27)) (justify left))
     )
-    (property "Footprint" "Relay_THT:Relay_1P1T_NO_10x24x18.8mm_Panasonic_ADW11xxxxW_THT" (id 2) (at 219.075 137.16 0)
+    (property "Footprint" "Relay_THT:RELAY PANASONIC" (id 2) (at 219.075 137.16 0)
       (effects (font (size 1.27 1.27)) hide)
     )
@@
     )
     (path "/aa5abb0b-a1bf-4c32-aa1a-3c3fa7fcfd10"
-      (reference "K1") (unit 1) (value "ADW11") (footprint "Relay_THT:Relay_1P1T_NO_10x24x18.8mm_Panasonic_ADW11xxxxW_THT")
+      (reference "K1") (unit 1) (value "ADW11") (footprint "Relay_THT:RELAY PANASONIC")
     )
     (path "/54b6a8c0-56ff-425d-a569-3f64dc62b610"
-      (reference "R1") (unit 1) (value "R") (footprint "Resistor_THT:R_Axial_DIN0207_L6.3mm_D2.5mm_P10.16mm_Horizontal")
+      (reference "R1") (unit 1) (value "330") (footprint "Resistor_THT:R_Axial_DIN0207_L6.3mm_D2.5mm_P10.16mm_Horizontal")
+    )
+    (path "/7856fd3e-7cb2-4617-9f08-e93b38475b94"
+      (reference "R2") (unit 1) (value "120") (footprint "Resistor_THT:R_Axial_DIN0207_L6.3mm_D2.5mm_P10.16mm_Horizontal")
     )
     (path "/81cccd6c-7099-4977-93e7-544e11021b8b"
