File: ground station/pcb/kicad Project/estacion terrena.kicad_pcb (KiCad board)
At the start: 2 copper layers, 94 x 93.8 mm, 18 parts, among them J1 Micro-usb_lora, J10 IDC_STLINK, J11 IDC_CANSAT, J2 Parte izquierda lora, J3 parte derecha lora, J4 Breakouy_micro_usb, J7 POSITIVO_LED TESTIGO, K1 ADW11, SW1 SWITCH

Commit message: Actualización
Parts:
- added 120: 120, Resistor_THT:R_Axial_DIN0207_L6.3mm_D2.5mm_P10.16mm_Horizontal, F.Cu at (169.1, 70.5)
- added GND: TestPoint_THTPad_D1.5mm_Drill0.7mm, TestPoint:TestPoint_THTPad_D1.5mm_Drill0.7mm, F.Cu at (168.0, 62.5)
- 330: renamed from R1; value R -> 330
- IDC CANSAT: renamed from J11
- IDC STLINK: renamed from J10
- RELAY: renamed from K1; footprint Relay_THT:Relay_1P1T_NO_10x24x18.8mm_Panasonic_ADW11xxxxW_THT -> Relay_THT:RELAY PANASONIC
- moved RELAY 16.7 mm to (164.5, 77.5), turned to 0 degrees
- moved J2 2.30 mm to (163.1, 109.7)
- moved J3 2.30 mm to (154.0, 131.7)
- moved REF** 1.00 mm to (128.5, 68.0)
- moved REF** 1.00 mm to (128.5, 101.5)
- moved REF** 1.00 mm to (128.5, 82.0)
- moved REF** 1.00 mm to (128.5, 87.5)
- renumbered J7 to LED+
Connections:
- 330 pad 2: Net-(K1-Pad1) -> Net-(R1-Pad2)
- SW1 pad 1: Net-(K1-Pad1) -> Net-(R1-Pad2)
Routing:
- net Net-(K1-Pad1): track 90.1 -> 4.48 mm
- net Net-(R1-Pad2): track 0.00 -> 80.9 mm
- net GND: track 124.0 -> 171.3 mm, vias 0 -> 2
- net /GNDBAT2: track 41.6 -> 54.4 mm
- net /VBAT1: track 83.1 -> 86.1 mm
- net /VCC_SW: track 37.0 -> 39.4 mm
- net GND1: track 63.9 -> 63.1 mm
Other:
- board text added: "GND"
- board text added: "RX"
- board text added: "TX"
- board text added: "VCC"

Commit message: Modificaciones
Parts:
- moved REF** 67.4 mm to (154.0, 130.3), turned to -120 degrees
- moved REF** 66.9 mm to (166.2, 137.3), turned to -120 degrees
- moved J1 61.0 mm to (153.4, 66.9), turned to -130 degrees
- moved J2 53.2 mm to (135.9, 63.9), turned to -40 degrees
- moved SW1 48.2 mm to (165.6, 79.1), turned to -120 degrees
- moved J3 47.2 mm to (147.0, 85.0), turned to -40 degrees
- moved REF** 44.2 mm to (168.1, 111.9), turned to -120 degrees
- moved J4 43.8 mm to (173.6, 73.3), turned to -125 degrees
- moved REF** 43.8 mm to (175.1, 115.9), turned to -120 degrees
- moved REF** 42.0 mm to (127.3, 129.5), turned to -120 degrees
- moved REF** 36.7 mm to (139.5, 136.5), turned to -120 degrees
- moved RELAY 26.9 mm to (148.3, 99.0), turned to 70 degrees
- moved LED+ 23.2 mm to (183.3, 74.9), turned to 80 degrees
- moved REF** 22.9 mm to (141.4, 111.1), turned to -120 degrees
- moved 330 21.5 mm to (179.3, 75.4), turned to -130 degrees
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Routing:
- net VCC: track 91.9 -> 27.5 mm
- net Net-(R1-Pad2): track 80.9 -> 19.0 mm
- net /VCC_SW: track 39.4 -> 85.8 mm, vias 0 -> 2
- net GND: track 171.3 -> 207.6 mm, vias 2 -> 0
- net /VBAT2: track 12.1 -> 48.4 mm
- net /GNDBAT2: track 54.4 -> 33.1 mm
- net /VBAT1: track 86.1 -> 66.1 mm
- net Net-(K1-Pad1): track 4.48 -> 19.0 mm
- net /RX: track 10.8 -> 22.5 mm
- net /SDIO_STL: track 28.0 -> 38.8 mm
- net /TX: track 11.4 -> 21.6 mm
- net GND1: track 63.1 -> 52.9 mm, vias 3 -> 0
- net /NC: track 11.9 -> 21.3 mm
- net /SCLK _STL_LINK: track 25.5 -> 19.1 mm
- net /LED: track 5.74 -> 4.25 mm
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
Commit message: ACTUALIZACION Y RERUTEO DE PLACA
Parts:
- moved REF** 77.6 mm to (119.2, 75.6), turned to 90 degrees
- moved J2 68.5 mm to (178.5, 117.6), turned to 175 degrees
- moved J4 66.4 mm to (155.1, 137.1), turned to 123 degrees
- moved IDC STLINK 61.3 mm to (143.1, 138.7), turned to -123 degrees
- moved REF** 60.7 mm to (138.7, 75.8), turned to 90 degrees
- moved REF** 59.3 mm to (152.7, 75.8), turned to 90 degrees
- moved J1 59.0 mm to (162.5, 125.2), turned to 85 degrees
- moved REF** 58.5 mm to (133.2, 75.6), turned to 90 degrees
- moved REF** 55.6 mm to (122.2, 98.6), turned to 90 degrees
- moved LED+ 53.3 mm to (131.4, 62.8), turned to 90 degrees
- moved GND 49.8 mm to (131.0, 69.0)
- moved 330 45.0 mm to (136.0, 63.1), turned to 0 degrees
- moved 120 43.8 mm to (113.4, 90.8), turned to -80 degrees
- moved IDC CANSAT 40.7 mm to (132.6, 123.5), turned to 90 degrees
- moved REF** 40.2 mm to (130.2, 98.6), turned to 90 degrees
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Routing:
- net /VCC_SW: track 85.8 -> 27.5 mm, vias 2 -> 0
- net VCC: track 27.5 -> 85.5 mm
- net Net-(R1-Pad2): track 19.0 -> 59.0 mm
- net /VBAT1: track 66.1 -> 44.4 mm, vias 0 -> 2
- net /VBAT2: track 48.4 -> 28.2 mm
- net GND1: track 52.9 -> 69.0 mm
- net Net-(K1-Pad1): track 19.0 -> 4.41 mm
- net GND: track 207.6 -> 194.9 mm, vias 0 -> 2
- net /NC: track 21.3 -> 10.7 mm
- net /GNDBAT2: track 33.1 -> 43.2 mm
- net /TX: track 21.6 -> 12.1 mm
- net /RX: track 22.5 -> 13.5 mm
- net /SDIO_STL: track 38.8 -> 47.5 mm
- net /VCC_STLINK: track 20.1 -> 14.8 mm
- net /SCLK _STL_LINK: track 19.1 -> 23.7 mm
Other:
- board text added: "Medio"
