File: ground station/pcb/Auxiliar_pcb/Pcb_auxiliar/Pcb_auxiliar.kicad_pcb (KiCad board)
At the start: 2 copper layers, 61.1 x 18 mm, 7 parts, among them J1 Conn_01x04_Male, J2 Conn_01x03_Male, SW1 SW_DPDT_x2

Commit message: Actualizaciones
Parts:
- D1: value LED_RGBK -> LED_RGBA
- moved R3 10.7 mm to (138.3, 87.0)
- moved R2 4.79 mm to (139.1, 89.2), turned to 20 degrees
- moved D1 4.70 mm to (146.7, 85.9), turned to -90 degrees
- moved R1 4.52 mm to (134.9, 92.3), turned to 0 degrees
Connections:
- net GND renamed Net-(J1-Pad4)
- R1 pad 1: Net-(J1-Pad1) -> Net-(J1-Pad3)
- R3 pad 1: Net-(J1-Pad3) -> Net-(J1-Pad1)
Routing:
- net Net-(R3-Pad2): track 14.6 -> 7.83 mm
- net Net-(R1-Pad2): track 5.94 -> 12.4 mm
- net Net-(J1-Pad2): track 3.51 -> 6.96 mm
- net Net-(R2-Pad2): track 10.0 -> 7.45 mm
- net Net-(J1-Pad3): track 3.91 -> 4.69 mm
