File: ground station/pcb/Auxiliar_pcb/Pcb_auxiliar/Pcb_auxiliar.kicad_sch (KiCad schematic)
At the start: 7 parts, among them J1 Conn_01x04_Male, J2 Conn_01x03_Male, SW1 SW_DPDT_x2

Commit message: Actualizaciones
Parts:
- removed D1: LED_RGBK, LED_THT:LED_D5.0mm-4_RGB, symbol Device:LED_RGBK
- added D1: LED_RGBA, LED_THT:LED_D5.0mm-4_RGB, symbol Device:LED_RGBA
Connections:
- net at J1.1 (Pin_1): now also R3.1; no longer R1.1
- net at J1.3 (Pin_3): now also R1.1; no longer R3.1
- net at R3.2: now also D1.1 (RK)
- net at R2.2: now also D1.2 (GK)
- net at R1.2: now also D1.3 (BK)
- net GND: no longer names the net of J1.4 (Pin_4)
- net GND: now also D1.4 (A)
Other:
- moved on the sheet: J1
Changed lines of the file:
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@@
 (kicad_sch (version 20211123) (generator eeschema)
   (paper "A4")
-  (junction (at 125.73 90.17) (diameter 0) (color 0 0 0 0)
-  )
   (polyline (pts (xy 152.4 55.88) (xy 152.4 102.87))
     (stroke (width 0) (type default) (color 0 0 0 0))
@@
     (stroke (width 0) (type default) (color 0 0 0 0))
   )
-  (wire (pts (xy 125.73 90.17) (xy 144.78 90.17))
-    (stroke (width 0) (type default) (color 0 0 0 0))
-  )
-  (wire (pts (xy 144.78 90.17) (xy 144.78 80.01))
-    (stroke (width 0) (type default) (color 0 0 0 0))
-  )
-  (wire (pts (xy 107.95 83.82) (xy 107.95 90.17))
+  (wire (pts (xy 107.95 62.23) (xy 144.78 62.23))
+    (stroke (width 0) (type default) (color 0 0 0 0))
+  )
+  (wire (pts (xy 144.78 62.23) (xy 144.78 80.01))
     (stroke (width 0) (type default) (color 0 0 0 0))
   )
@@
     (stroke (width 0) (type default) (color 0 0 0 0))
   )
+  (wire (pts (xy 107.95 62.23) (xy 107.95 73.66))
+    (stroke (width 0) (type default) (color 0 0 0 0))
+  )
   (wire (pts (xy 203.2 80.01) (xy 200.66 80.01))
     (stroke (width 0) (type default) (color 0 0 0 0))
@@
   )
   (wire (pts (xy 172.72 85.09) (xy 182.88 85.09))
-    (stroke (width 0) (type default) (color 0 0 0 0))
-  )
-  (wire (pts (xy 107.95 90.17) (xy 125.73 90.17))
-    (stroke (width 0) (type default) (color 0 0 0 0))
-  )
-  (wire (pts (xy 125.73 90.17) (xy 125.73 93.98))
     (stroke (width 0) (type default) (color 0 0 0 0))
   )
@@
     (effects (font (size 1.27 1.27)) (justify left bottom))
   )
-  (symbol (lib_id "Connector:Conn_01x04_Male") (at 102.87 78.74 0) (unit 1)
-    (in_bom yes) (on_board yes) (fields_autoplaced)
-    (property "Reference" "J1" (id 0) (at 103.505 71.12 0))
-    (property "Value" "Conn_01x04_Male" (id 1) (at 103.505 73.66 0))
+  (symbol (lib_id "Connector:Conn_01x04_Male") (at 102.87 78.74 0) (mirror x) (unit 1)
+    (in_bom yes) (on_board yes) (fields_autoplaced)
+    (property "Reference" "J1" (id 0) (at 101.6 76.1999 0)
+      (effects (font (size 1.27 1.27)) (justify right))
+    )
+    (property "Value" "Conn_01x04_Male" (id 1) (at 101.6 78.7399 0)
+      (effects (font (size 1.27 1.27)) (justify right))
+    )
     (property "Footprint" "Connector_PinSocket_2.54mm:PinSocket_1x04_P2.54mm_Vertical" (id 2) (at 102.87 78.74 0)
       (effects (font (size 1.27 1.27)) hide)
@@
     (pin "3")
     (pin "4")
-  )
-  (symbol (lib_id "power:GND") (at 125.73 93.98 0) (unit 1)
-    (in_bom yes) (on_board yes) (fields_autoplaced)
-    (property "Reference" "#PWR01" (id 0) (at 125.73 100.33 0)
-      (effects (font (size 1.27 1.27)) hide)
-    )
-    (property "Value" "GND" (id 1) (at 125.73 99.06 0))
-    (property "Footprint" "" (id 2) (at 125.73 93.98 0)
-      (effects (font (size 1.27 1.27)) hide)
-    )
-    (property "Datasheet" "" (id 3) (at 125.73 93.98 0)
-      (effects (font (size 1.27 1.27)) hide)
-    )
-    (pin "1")
   )
   (symbol (lib_id "Connector:Conn_01x03_Male") (at 167.64 82.55 0) (unit 1)
@@
     (pin "2")
   )
-  (symbol (lib_id "Device:LED_RGBK") (at 139.7 80.01 180) (unit 1)
-    (in_bom yes) (on_board yes)
-    (property "Reference" "D1" (id 0) (at 139.7 66.04 0))
-    (property "Value" "LED_RGBK" (id 1) (at 139.7 69.85 0))
+  (symbol (lib_id "Device:LED_RGBA") (at 139.7 80.01 0) (mirror x) (unit 1)
+    (in_bom yes) (on_board yes) (fields_autoplaced)
+    (property "Reference" "D1" (id 0) (at 139.7 67.31 0))
+    (property "Value" "LED_RGBA" (id 1) (at 139.7 69.85 0))
     (property "Footprint" "LED_THT:LED_D5.0mm-4_RGB" (id 2) (at 139.7 78.74 0)
       (effects (font (size 1.27 1.27)) hide)
@@
   )
   (symbol_instances
-    (path "/4bcafdc8-5e44-471d-8059-c4f31964f976"
-      (reference "#PWR01") (unit 1) (value "GND") (footprint "")
-    )
-    (path "/87af33f3-41a3-4b5e-aeeb-0ac6403351ff"
-      (reference "D1") (unit 1) (value "LED_RGBK") (footprint "LED_THT:LED_D5.0mm-4_RGB")
+    (path "/79bd839b-cf80-4141-bdfb-75c9776513c5"
+      (reference "D1") (unit 1) (value "LED_RGBA") (footprint "LED_THT:LED_D5.0mm-4_RGB")
     )
     (path "/3eb34af4-da13-4e59-8401-9125bfa36c5b"
