File: ground station/pcb/PCB_GS/estacion terrena.kicad_sch (KiCad schematic)
At the start: 15 parts, among them J1 Micro-usb_lora, J10 IDC_STLINK, J11 IDC_CANSAT, J2 Parte izquierda lora, J3 parte derecha lora, J4 Breakouy_micro_usb, J5 CARG_BAT_1_OUT, J6 CARG_BAT_1_IN, J7 POSITIVO_LED TESTIGO, J8 CARG_BAT_2_OUT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

Commit message: Adición de modificaciones y nuevo diseño de placa
Parts:
- added J12: LED_CARGA_1, Connector_Pin:Pin_D1.0mm_L10.0mm, symbol Connector:Conn_01x01_Female
- added J13: LED_CARGA_2, Connector_Pin:Pin_D1.0mm_L10.0mm, symbol Connector:Conn_01x01_Female
- added J14: conector RGB, Connector_PinSocket_2.54mm:PinSocket_1x04_P2.54mm_Vertical, symbol Connector:Conn_01x04_Female
- added R3, R4: 10K, Resistor_SMD:R_0805_2012Metric_Pad1.20x1.40mm_HandSolder, symbol Device:R
Connections:
- net GND: now also J14.4 (Pin_4), R3.1, R4.1
- net LED_CARGA_1: now reaches J3.5 (Pin_5)
- net LED_CARGA_1: now also J12.1 (Pin_1), R3.2
- net LED_CARGA_2: now reaches J3.6 (Pin_6)
- net LED_CARGA_2: now also J13.1 (Pin_1), R4.2
- net R: now reaches J3.7 (Pin_7)
- net R: now also J14.1 (Pin_1)
- net G: now reaches J3.8 (Pin_8)
- net G: now also J14.2 (Pin_2)
- net B: now reaches J3.9 (Pin_9)
- net B: now also J14.3 (Pin_3)
- no-connect marks 38 -> 33
Other:
- note added: "RESISTENCIAS PULL DOWN ENTRADAS LORA"

Commit message: Actualizaciones
Parts:
- added R5: 10K, Resistor_SMD:R_0805_2012Metric_Pad1.20x1.40mm_HandSolder, symbol Device:R
Connections:
- net GND: now also R5.2; no longer J14.4 (Pin_4)
- net VCC: now also J14.4 (Pin_4)
- net VCC_SW: now also J3.11 (Pin_11), R5.1
- no-connect marks 33 -> 32
Changed lines of the file:
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@@
   (no_connect (at 99.06 95.25))
   (no_connect (at 124.46 97.79))
-  (no_connect (at 124.46 95.25))
   (no_connect (at 124.46 92.71))
   (no_connect (at 124.46 77.47))
@@
     (stroke (width 0) (type default) (color 0 0 0 0))
   )
-  (wire (pts (xy 214.63 121.92) (xy 213.36 121.92))
+  (wire (pts (xy 214.63 114.3) (xy 213.36 114.3))
     (stroke (width 0) (type default) (color 0 0 0 0))
   )
@@
     (stroke (width 0) (type default) (color 0 0 0 0))
   )
+  (wire (pts (xy 194.31 44.45) (xy 194.31 46.99))
+    (stroke (width 0) (type default) (color 0 0 0 0))
+  )
   (wire (pts (xy 156.21 138.43) (xy 157.48 138.43))
     (stroke (width 0) (type default) (color 0 0 0 0))
@@
     (stroke (width 0) (type default) (color 0 0 0 0))
   )
-  (polyline (pts (xy 146.05 29.21) (xy 185.42 29.21))
+  (polyline (pts (xy 146.05 29.21) (xy 209.55 29.21))
     (stroke (width 0) (type default) (color 0 0 0 0))
   )
@@
     (stroke (width 0) (type default) (color 0 0 0 0))
   )
-  (polyline (pts (xy 185.42 54.61) (xy 146.05 54.61))
+  (polyline (pts (xy 209.55 54.61) (xy 146.05 54.61))
+    (stroke (width 0) (type default) (color 0 0 0 0))
+  )
+  (wire (pts (xy 213.36 111.76) (xy 213.36 114.3))
     (stroke (width 0) (type default) (color 0 0 0 0))
   )
@@
     (stroke (width 0) (type default) (color 0 0 0 0))
   )
-  (wire (pts (xy 213.36 121.92) (xy 213.36 127))
-    (stroke (width 0) (type default) (color 0 0 0 0))
-  )
   (wire (pts (xy 180.34 143.51) (xy 180.34 147.32))
     (stroke (width 0) (type default) (color 0 0 0 0))
@@
     (stroke (width 0) (type default) (color 0 0 0 0))
   )
-  (polyline (pts (xy 185.42 29.21) (xy 185.42 54.61))
+  (polyline (pts (xy 209.55 29.21) (xy 209.55 54.61))
     (stroke (width 0) (type default) (color 0 0 0 0))
   )
@@
     (effects (font (size 1.27 1.27)) (justify left bottom))
   )
-  (label "B" (at 214.63 119.38 0)
+  (label "B" (at 214.63 116.84 0)
     (effects (font (size 1.27 1.27)) (justify left bottom))
   )
@@
     (effects (font (size 1.27 1.27)) (justify right bottom))
   )
+  (label "VCC_SW" (at 194.31 36.83 0)
+    (effects (font (size 1.27 1.27)) (justify left bottom))
+  )
   (label "GNDBAT1" (at 207.01 68.58 180)
     (effects (font (size 1.27 1.27)) (justify right bottom))
   )
-  (label "R" (at 214.63 114.3 0)
+  (label "R" (at 214.63 121.92 0)
     (effects (font (size 1.27 1.27)) (justify left bottom))
   )
@@
     (effects (font (size 1.27 1.27)) (justify left bottom))
   )
-  (label "G" (at 214.63 116.84 0)
+  (label "G" (at 214.63 119.38 0)
     (effects (font (size 1.27 1.27)) (justify left bottom))
   )
@@
   (label "VBAT2" (at 173.99 95.25 270)
     (effects (font (size 1.27 1.27)) (justify right bottom))
+  )
+  (label "VCC_SW" (at 124.46 95.25 0)
+    (effects (font (size 1.27 1.27)) (justify left bottom))
   )
   (label "GNDBAT1" (at 152.4 95.25 270)
@@
     (pin "5")
   )
-  (symbol (lib_id "power:GND") (at 213.36 127 0) (unit 1)
-    (in_bom yes) (on_board yes) (fields_autoplaced)
-    (property "Reference" "#PWR011" (id 0) (at 213.36 133.35 0)
-      (effects (font (size 1.27 1.27)) hide)
-    )
-    (property "Value" "GND" (id 1) (at 213.36 132.08 0))
-    (property "Footprint" "" (id 2) (at 213.36 127 0)
-      (effects (font (size 1.27 1.27)) hide)
-    )
-    (property "Datasheet" "" (id 3) (at 213.36 127 0)
-      (effects (font (size 1.27 1.27)) hide)
-    )
-    (pin "1")
-  )
   (symbol (lib_id "Device:R") (at 171.45 40.64 180) (unit 1)
     (in_bom yes) (on_board yes) (fields_autoplaced)
@@
     (pin "2")
   )
+  (symbol (lib_id "power:VCC") (at 213.36 111.76 0) (unit 1)
+    (in_bom yes) (on_board yes) (fields_autoplaced)
+    (property "Reference" "#PWR?" (id 0) (at 213.36 115.57 0)
+      (effects (font (size 1.27 1.27)) hide)
+    )
+    (property "Value" "VCC" (id 1) (at 213.36 106.68 0))
+    (property "Footprint" "" (id 2) (at 213.36 111.76 0)
+      (effects (font (size 1.27 1.27)) hide)
+    )
+    (property "Datasheet" "" (id 3) (at 213.36 111.76 0)
+      (effects (font (size 1.27 1.27)) hide)
+    )
+    (pin "1")
+  )
   (symbol (lib_id "Connector:Conn_01x04_Female") (at 173.99 90.17 90) (unit 1)
     (in_bom yes) (on_board yes) (fields_autoplaced)
@@
     (pin "4")
   )
+  (symbol (lib_id "Device:R") (at 194.31 40.64 0) (unit 1)
+    (in_bom yes) (on_board yes) (fields_autoplaced)
+    (property "Reference" "R5" (id 0) (at 196.85 39.3699 0)
+      (effects (font (size 1.27 1.27)) (justify left))
+    )
+    (property "Value" "10K" (id 1) (at 196.85 41.9099 0)
+      (effects (font (size 1.27 1.27)) (justify left))
+    )
+    (property "Footprint" "Resistor_SMD:R_0805_2012Metric_Pad1.20x1.40mm_HandSolder" (id 2) (at 192.532 40.64 90)
+      (effects (font (size 1.27 1.27)) hide)
+    )
+    (property "Datasheet" "~" (id 3) (at 194.31 40.64 0)
+      (effects (font (size 1.27 1.27)) hide)
+    )
+    (pin "1")
+    (pin "2")
+  )
   (symbol (lib_id "power:PWR_FLAG") (at 109.22 35.56 180) (unit 1)
     (in_bom yes) (on_board yes) (fields_autoplaced)
@@
     )
     (property "Datasheet" "" (id 3) (at 109.22 27.94 0)
+      (effects (font (size 1.27 1.27)) hide)
+    )
+    (pin "1")
+  )
+  (symbol (lib_id "power:GND") (at 194.31 46.99 0) (unit 1)
+    (in_bom yes) (on_board yes) (fields_autoplaced)
+    (property "Reference" "#PWR014" (id 0) (at 194.31 53.34 0)
+      (effects (font (size 1.27 1.27)) hide)
+    )
+    (property "Value" "GND" (id 1) (at 194.31 52.07 0))
+    (property "Footprint" "" (id 2) (at 194.31 46.99 0)
+      (effects (font (size 1.27 1.27)) hide)
+    )
+    (property "Datasheet" "" (id 3) (at 194.31 46.99 0)
       (effects (font (size 1.27 1.27)) hide)
     )
@@
     (pin "1")
   )
-  (symbol (lib_id "Connector:Conn_01x04_Female") (at 219.71 116.84 0) (unit 1)
-    (in_bom yes) (on_board yes) (fields_autoplaced)
-    (property "Reference" "J14" (id 0) (at 220.98 116.8399 0)
-      (effects (font (size 1.27 1.27)) (justify left))
-    )
-    (property "Value" "conector RGB" (id 1) (at 220.98 119.3799 0)
-      (effects (font (size 1.27 1.27)) (justify left))
-    )
-    (property "Footprint" "Connector_PinSocket_2.54mm:PinSocket_1x04_P2.54mm_Vertical" (id 2) (at 219.71 116.84 0)
-      (effects (font (size 1.27 1.27)) hide)
-    )
-    (property "Datasheet" "~" (id 3) (at 219.71 116.84 0)
+  (symbol (lib_id "Connector:Conn_01x04_Female") (at 219.71 119.38 0) (mirror x) (unit 1)
+    (in_bom yes) (on_board yes) (fields_autoplaced)
+    (property "Reference" "J14" (id 0) (at 220.98 119.3801 0)
+      (effects (font (size 1.27 1.27)) (justify left))
+    )
+    (property "Value" "conector RGB" (id 1) (at 220.98 116.8401 0)
+      (effects (font (size 1.27 1.27)) (justify left))
+    )
+    (property "Footprint" "Connector_PinSocket_2.54mm:PinSocket_1x04_P2.54mm_Vertical" (id 2) (at 219.71 119.38 0)
+      (effects (font (size 1.27 1.27)) hide)
+    )
+    (property "Datasheet" "~" (id 3) (at 219.71 119.38 0)
       (effects (font (size 1.27 1.27)) hide)
     )
@@
       (reference "#PWR010") (unit 1) (value "GND") (footprint "")
     )
-    (path "/2b47e5ee-c95c-498a-a97d-19fbb2cc2449"
-      (reference "#PWR011") (unit 1) (value "GND") (footprint "")
-    )
     (path "/158f9dee-ec88-45b7-84c9-97fc4e158b08"
       (reference "#PWR012") (unit 1) (value "GND") (footprint "")
@@
       (reference "#PWR013") (unit 1) (value "GND") (footprint "")
     )
+    (path "/95054fa1-06d5-4985-902e-0fe03894165c"
+      (reference "#PWR014") (unit 1) (value "GND") (footprint "")
+    )
+    (path "/67f1aadd-abbf-42af-b69d-c0bc8ff3c54d"
+      (reference "#PWR?") (unit 1) (value "VCC") (footprint "")
+    )
     (path "/28f1f78a-2a0e-408c-8286-8740eff044c4"
       (reference "J1") (unit 1) (value "Micro-usb_lora") (footprint "Connector_PinSocket_2.00mm:PinSocket_1x05_P2.00mm_Vertical")
@@
       (reference "R4") (unit 1) (value "10K") (footprint "Resistor_SMD:R_0805_2012Metric_Pad1.20x1.40mm_HandSolder")
     )
+    (path "/86365ce4-1f78-4d23-9f4f-d288db7fffab"
+      (reference "R5") (unit 1) (value "10K") (footprint "Resistor_SMD:R_0805_2012Metric_Pad1.20x1.40mm_HandSolder")
+    )
     (path "/81cccd6c-7099-4977-93e7-544e11021b8b"

Commit message: Actualizacion
Parts:
- removed J7: POSITIVO_LED TESTIGO, Connector_Pin:Pin_D0.9mm_L10.0mm_W2.4mm_FlatFork, symbol Connector:Conn_01x01_Female
- removed R1: 330, Resistor_THT:R_Axial_DIN0207_L6.3mm_D2.5mm_P10.16mm_Horizontal, symbol Device:R
Changed lines of the file:
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@@
   (junction (at 163.83 67.31) (diameter 0) (color 0 0 0 0)
-  )
-  (junction (at 167.64 128.27) (diameter 0) (color 0 0 0 0)
   )
   (junction (at 105.41 121.92) (diameter 0) (color 0 0 0 0)
@@
     (stroke (width 0) (type default) (color 0 0 0 0))
   )
-  (wire (pts (xy 156.21 128.27) (xy 167.64 128.27))
-    (stroke (width 0) (type default) (color 0 0 0 0))
-  )
   (wire (pts (xy 134.62 80.01) (xy 134.62 83.82))
     (stroke (width 0) (type default) (color 0 0 0 0))
@@
     (stroke (width 0) (type default) (color 0 0 0 0))
   )
-  (wire (pts (xy 167.64 125.73) (xy 167.64 128.27))
-    (stroke (width 0) (type default) (color 0 0 0 0))
-  )
   (wire (pts (xy 134.62 83.82) (xy 138.43 83.82))
     (stroke (width 0) (type default) (color 0 0 0 0))
@@
     (stroke (width 0) (type default) (color 0 0 0 0))
   )
-  (wire (pts (xy 167.64 115.57) (xy 167.64 118.11))
-    (stroke (width 0) (type default) (color 0 0 0 0))
-  )
   (polyline (pts (xy 135.89 60.96) (xy 135.89 106.68))
     (stroke (width 0) (type default) (color 0 0 0 0))
@@
     (stroke (width 0) (type default) (color 0 0 0 0))
   )
-  (wire (pts (xy 167.64 128.27) (xy 170.18 128.27))
+  (wire (pts (xy 156.21 128.27) (xy 170.18 128.27))
     (stroke (width 0) (type default) (color 0 0 0 0))
   )
@@
   )
   (label "GND" (at 105.41 132.08 0)
-    (effects (font (size 1.27 1.27)) (justify left bottom))
-  )
-  (label "LED" (at 167.64 118.11 0)
     (effects (font (size 1.27 1.27)) (justify left bottom))
   )
@@
     (pin "1")
   )
-  (symbol (lib_id "Device:R") (at 167.64 121.92 0) (unit 1)
-    (in_bom yes) (on_board yes)
-    (property "Reference" "R1" (id 0) (at 170.18 120.6499 0)
-      (effects (font (size 1.27 1.27)) (justify left))
-    )
-    (property "Value" "330" (id 1) (at 162.56 121.92 0)
-      (effects (font (size 1.27 1.27)) (justify left))
-    )
-    (property "Footprint" "Resistor_THT:R_Axial_DIN0207_L6.3mm_D2.5mm_P10.16mm_Horizontal" (id 2) (at 165.862 121.92 90)
-      (effects (font (size 1.27 1.27)) hide)
-    )
-    (property "Datasheet" "~" (id 3) (at 167.64 121.92 0)
-      (effects (font (size 1.27 1.27)) hide)
-    )
-    (pin "1")
-    (pin "2")
-  )
   (symbol (lib_id "power:VCC") (at 213.36 111.76 0) (unit 1)
     (in_bom yes) (on_board yes) (fields_autoplaced)
@@
     (pin "1")
   )
-  (symbol (lib_id "Connector:Conn_01x01_Female") (at 167.64 110.49 90) (unit 1)
-    (in_bom yes) (on_board yes) (fields_autoplaced)
-    (property "Reference" "J7" (id 0) (at 168.91 109.8549 90)
-      (effects (font (size 1.27 1.27)) (justify right))
-    )
-    (property "Value" "POSITIVO_LED TESTIGO" (id 1) (at 168.91 112.3949 90)
-      (effects (font (size 1.27 1.27)) (justify right))
-    )
-    (property "Footprint" "Connector_Pin:Pin_D0.9mm_L10.0mm_W2.4mm_FlatFork" (id 2) (at 167.64 110.49 0)
-      (effects (font (size 1.27 1.27)) hide)
-    )
-    (property "Datasheet" "~" (id 3) (at 167.64 110.49 0)
-      (effects (font (size 1.27 1.27)) hide)
-    )
-    (pin "1")
-  )
   (symbol (lib_id "Connector:Conn_01x04_Female") (at 219.71 119.38 0) (mirror x) (unit 1)
     (in_bom yes) (on_board yes) (fields_autoplaced)
@@
       (reference "J6") (unit 1) (value "CARG_BAT_1_IN") (footprint "")
     )
-    (path "/dc594fb9-a1c4-4628-95bf-9bebd0c4fd80"
-      (reference "J7") (unit 1) (value "POSITIVO_LED TESTIGO") (footprint "Connector_Pin:Pin_D0.9mm_L10.0mm_W2.4mm_FlatFork")
-    )
     (path "/68da8cc6-0765-4da4-9976-d371a52df850"
       (reference "J8") (unit 1) (value "CARG_BAT_2_OUT") (footprint "")
@@
       (reference "K1") (unit 1) (value "ADW11") (footprint "Relay_THT:RELAY PANASONIC")
     )
-    (path "/54b6a8c0-56ff-425d-a569-3f64dc62b610"
-      (reference "R1") (unit 1) (value "330") (footprint "Resistor_THT:R_Axial_DIN0207_L6.3mm_D2.5mm_P10.16mm_Horizontal")
-    )
     (path "/7856fd3e-7cb2-4617-9f08-e93b38475b94"
